File: sensorbox-battery-powered.sch (KiCad schematic (older format))
At the start: 17 parts, among them J1 Conn_01x02, J2 Conn_01x06_Male, SW1 Reset, SW2 Program, U1 ESP-12F, U2 BME280

Commit message: Add battery sensing circuit.
Parts:
- added Q1: AO3401A, Package_TO_SOT_SMD:SOT-23, symbol Transistor_FET:AO3401A
- added R6: 33k, Resistor_SMD:R_0805_2012Metric, symbol Device:R
- added R7, R8: 10k, Resistor_SMD:R_0805_2012Metric, symbol Device:R
Connections:
- net GND: now also R7.2
- net BAT_SENS: now reaches U1.2 (ADC)
- net BAT_SENS: now also R6.2, R7.1
- net ENABLE_BAT_SENS: now reaches U1.5 (GPIO14)
- net ENABLE_BAT_SENS: now also Q1.1 (G), R8.2
- net +BATT: now reaches C4.1, J1.1 (Pin_1), L1.2 (VIN)
- net +BATT: now also Q1.2 (S), R8.1
- new net: Q1.3 (D), R6.1
- no-connect marks 12 -> 11
Other:
- moved on the sheet: C1, R1, R2, SW1

Commit message: Use SMD battery connector.
Parts:
- J1: footprint Connector_JST:JST_PH_S2B-PH-K_1x02_P2.00mm_Horizontal -> jst-conectors:JST_PH_S2B-PH-SM4-TB_1x02-1MP_P2.00mm_Horizontal; LCSC (none) -> C295747
Changed lines of the file:
@@
 	4500 5700 4500 5550
 Connection ~ 4500 5550
-$Comp
-L Connector_Generic:Conn_01x02 J1
-U 1 1 62BC16F6
-P 2950 5400
-F 0 "J1" H 2868 5075 50  0000 C CNN
-F 1 "Conn_01x02" H 2868 5166 50  0000 C CNN
-F 2 "Connector_JST:JST_PH_S2B-PH-K_1x02_P2.00mm_Horizontal" H 2950 5400 50  0001 C CNN
-F 3 "~" H 2950 5400 50  0001 C CNN
-	1    2950 5400
-	-1   0    0    1
-$EndComp
 Wire Wire Line
 	3750 5550 3400 5550
@@
 	9650 4300 9500 4300
 Connection ~ 9500 4300
+$Comp
+L Connector_Generic:Conn_01x02 J1
+U 1 1 62BC16F6
+P 2950 5400
+F 0 "J1" H 2868 5075 50  0000 C CNN
+F 1 "Conn_01x02" H 2868 5166 50  0000 C CNN
+F 2 "jst-conectors:JST_PH_S2B-PH-SM4-TB_1x02-1MP_P2.00mm_Horizontal" H 2950 5400 50  0001 C CNN
+F 3 "~" H 2950 5400 50  0001 C CNN
+F 4 "C295747" H 2950 5400 50  0001 C CNN "LCSC"
+	1    2950 5400
+	-1   0    0    1
+$EndComp
 $EndSCHEMATC
