File: hardware/battery-powered/sensorbox-battery-powered.kicad_pcb (KiCad board)
At the start: 2 copper layers, 30 x 55 mm, 25 parts, among them J1 Conn_01x02, J2 Conn_01x06_Male, Q1 AO3401A, SW1 Reset, SW2 Program, U1 ESP-12F, U2 BME280

Commit message: Remove JST connectors libraries.
Parts:
- J1: footprint jst-conectors:JST_PH_S2B-PH-SM4-TB_1x02-1MP_P2.00mm_Horizontal -> Connector_JST:JST_PH_S2B-PH-SM4-TB_1x02-1MP_P2.00mm_Horizontal
Connections:
- net +3V3 renamed +3.3V
- J2 pad 2: Net-(J2-Pad2) -> unconnected-(J2-Pad2)
- J2 pad 3: Net-(J2-Pad3) -> unconnected-(J2-Pad3)
- J2 pad 6: Net-(J2-Pad6) -> unconnected-(J2-Pad6)
- U1 pad 17: Net-(U1-Pad17) -> unconnected-(U1-Pad17)
- U1 pad 18: Net-(U1-Pad18) -> unconnected-(U1-Pad18)
- U1 pad 19: Net-(U1-Pad19) -> unconnected-(U1-Pad19)
- U1 pad 20: Net-(U1-Pad20) -> unconnected-(U1-Pad20)
- U1 pad 21: Net-(U1-Pad21) -> unconnected-(U1-Pad21)
- U1 pad 22: Net-(U1-Pad22) -> unconnected-(U1-Pad22)
- U1 pad 6: Net-(U1-Pad6) -> unconnected-(U1-Pad6)
- U1 pad 7: Net-(U1-Pad7) -> unconnected-(U1-Pad7)
Routing:
- net Net-(C1-Pad2): track 75.7 -> 73.5 mm
- net Net-(C5-Pad2): track 63.9 -> 62.8 mm
- net +3.3V: track 0.70 -> 0.16 mm
- net Net-(R5-Pad2): track 13.4 -> 12.9 mm
Other:
- net class Default removed
