File: hardware/battery-powered/sensorbox-battery-powered.sch (KiCad schematic (older format))
At the start: 21 parts, among them J1 Conn_01x02, J2 Conn_01x06_Male, Q1 AO3401A, SW1 Reset, SW2 Program, U1 ESP-12F, U2 BME280

Commit message: Remove JST connectors libraries.
Parts:
- J1: footprint jst-conectors:JST_PH_S2B-PH-SM4-TB_1x02-1MP_P2.00mm_Horizontal -> Connector_JST:JST_PH_S2B-PH-SM4-TB_1x02-1MP_P2.00mm_Horizontal
- L1: symbol ht7333-a:HT7333-A -> sensorbox-battery-powered-rescue:HT7333-A-ht7333-a
- U1: symbol kicad-ESP8266:ESP-12F -> sensorbox-battery-powered-rescue:ESP-12F-kicad-ESP8266
Changed lines of the file:
@@
 $EndDescr
 $Comp
-L kicad-ESP8266:ESP-12F U1
+L sensorbox-battery-powered-rescue:ESP-12F-kicad-ESP8266 U1
 U 1 1 62B7796D
 P 5400 2850
@@
 	6300 2950 7100 2950
 $Comp
-L ht7333-a:HT7333-A L1
+L sensorbox-battery-powered-rescue:HT7333-A-ht7333-a L1
 U 1 1 62BB3C55
 P 4350 5100
@@
 F 0 "J1" H 2868 5075 50  0000 C CNN
 F 1 "Conn_01x02" H 2868 5166 50  0000 C CNN
-F 2 "jst-conectors:JST_PH_S2B-PH-SM4-TB_1x02-1MP_P2.00mm_Horizontal" H 2950 5400 50  0001 C CNN
+F 2 "Connector_JST:JST_PH_S2B-PH-SM4-TB_1x02-1MP_P2.00mm_Horizontal" H 2950 5400 50  0001 C CNN
 F 3 "~" H 2950 5400 50  0001 C CNN
 F 4 "C295747" H 2950 5400 50  0001 C CNN "LCSC"
